File: Digital BMS Slave board .brd (EAGLE design)
At the start: 100 x 60 mm, 236 parts, among them J1 S4B-PH-K, J10 S3B-PH-K, J11 S6B-PH-K, J12 S4B-PH-K, J2 S4B-PH-K, J3 S4B-PH-K, J4 S6B-PH-K, J5 S2B-PH-K, J6 S2B-PH-K, J7 S2B-PH-K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

Commit message: Full routing 1.0ver. to review
DRC rules checked
Parts:
- removed J4: S6B-PH-K, con-jst-ph:S6B-PH-K
- removed TP13, TP65, TP66, TP67, TP68, TP69, TP70: TEST_PAD-[1.27MM], testing:TP1.27MM
- added J13: MOLEX22-12-406205-7068, commonly used connectors:7395-06
- moved C59 11.0 mm to (52.1, 12.9), turned to 270 degrees
- moved D13 9.72 mm to (5.87, 36.8), turned to 90 degrees
- moved R46 9.29 mm to (42.5, 5.44)
- moved R100 8.61 mm to (97.9, 26.0)
- moved JP20 8.21 mm to (39.4, 8.49), turned to 90 degrees
- moved C68 8.14 mm to (61.7, 35.5)
- moved C64 8.10 mm to (65.6, 35.5)
- moved C60 8.10 mm to (69.5, 35.5)
- moved D10 7.02 mm to (5.87, 28.4)
- moved TP54 6.72 mm to (89.9, 19.2)
- moved R45 6.48 mm to (51.3, 5.44), turned to 180 degrees
- moved C57 6.22 mm to (46.1, 14.1)
- moved TP56 6.08 mm to (76.4, 19.2)
- moved C70 5.77 mm to (59.9, 37.5)
- moved C66 5.72 mm to (63.7, 37.5), turned to 0 degrees
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Connections:
- net CB0: no longer TP13.1
- net CB1: no longer TP70.1
- net CB2: no longer TP69.1
- net CB3: no longer TP68.1
- net CB4: no longer TP67.1
- net CB5: no longer TP66.1
- net CB6: no longer TP65.1
- net GND: now also J13.6; no longer J4.6
- net NFAULT: now also J13.5; no longer J4.5
- net RX1: now also J13.3; no longer J4.3
- net TX: now also J13.2; no longer J4.2
- net VIO: now also J13.4; no longer J4.1
- net WAKEUP: now also J13.1; no longer J4.4
Routing:
- net CB5: track 2.68 -> 118.6 mm, vias 1 -> 4
- net CB4: track 2.48 -> 112.0 mm, vias 1 -> 4
- net CB6: track 6.99 -> 107.9 mm
- net CB3: track 2.54 -> 103.4 mm, vias 1 -> 4
- net CB2: track 2.74 -> 99.4 mm, vias 1 -> 4
- net CB1: track 2.94 -> 92.7 mm, vias 1 -> 4
- net CB0: track 3.56 -> 86.7 mm, vias 0 -> 4
- net VCC: track 55.3 -> 102.2 mm
- net BAT5: track 26.9 -> 73.2 mm
- net BAT4: track 26.4 -> 67.5 mm
- net BAT3: track 26.5 -> 64.3 mm
- net BAT1: track 28.6 -> 63.5 mm
- net BAT2: track 26.4 -> 60.4 mm
- net EB0: track 2.91 -> 35.9 mm, vias 0 -> 2
- net VIO: track 35.8 -> 67.6 mm, vias 1 -> 5
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