File: Digital BMS Slave board .sch (EAGLE design)
At the start: 270 parts, among them J1 S4B-PH-K, J10 S3B-PH-K, J11 S6B-PH-K, J12 MOLEX22-12-406205-7068, J13 S2B-PH-K, J14 S2B-PH-K, J15 S6B-PH-K, J2 S4B-PH-K, J3 S4B-PH-K, J4 S4B-PH-K, J5 S2B-PH-K, J6 S2B-PH-K, J7 S2B-PH-K, J8 S2B-PH-K, J9 S3B-PH-K, Q1 BSS123, Q2 BSS123, Q3 BSS123, Q4 BSS123, Q5 BSS123, Q6 BSS123, SW1 5PIN-DIP-SWITCH, U1 BQ79606A-Q1-HTQFP|48|9VIA, U2 ISO7342, X1 PESD2CAN, X2 PESD2CAN, X3 PESD2CAN, X4 PESD2CAN

Commit message: Gerbers for first order
Parts:
- C28, C32, C42, C46: value 0.33u/16V -> 0.33u/50V
Other:
- note added: "fail in 100V cap voltage rating"
- note added: "fail in 50V cap voltage rating"
Changed lines of the file:
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@@
 <layer number="155" name="FabDoc3" color="7" fill="1" visible="yes" active="yes"/>
 <layer number="170" name="tAssembl" color="1" fill="1" visible="yes" active="yes"/>
-<layer number="171" name="bAssembl" color="23" fill="1" visible="no" active="yes"/>
+<layer number="171" name="bAssembl" color="23" fill="1" visible="yes" active="yes"/>
 <layer number="191" name="mNets" color="7" fill="1" visible="no" active="no"/>
 <layer number="192" name="mBusses" color="7" fill="1" visible="no" active="no"/>
@@
 <variant name="PC_Test_BOT" populate="no"/>
 </part>
-<part name="C28" library="Capacitors" library_urn="urn:adsk.eagle:library:13360199" deviceset="C-EU" device="0603" package3d_urn="urn:adsk.eagle:package:14720896/4" value="0.33u/16V">
-<variant name="Full_Assembly_BOT" populate="no"/>
-<variant name="PC_Test_BOT" populate="no"/>
-</part>
-<part name="C32" library="Capacitors" library_urn="urn:adsk.eagle:library:13360199" deviceset="C-EU" device="0603" package3d_urn="urn:adsk.eagle:package:14720896/4" value="0.33u/16V">
+<part name="C28" library="Capacitors" library_urn="urn:adsk.eagle:library:13360199" deviceset="C-EU" device="0603" package3d_urn="urn:adsk.eagle:package:14720896/4" value="0.33u/50V">
+<variant name="Full_Assembly_BOT" populate="no"/>
+<variant name="PC_Test_BOT" populate="no"/>
+</part>
+<part name="C32" library="Capacitors" library_urn="urn:adsk.eagle:library:13360199" deviceset="C-EU" device="0603" package3d_urn="urn:adsk.eagle:package:14720896/4" value="0.33u/50V">
 <variant name="Full_Assembly_BOT" populate="no"/>
 <variant name="PC_Test_BOT" populate="no"/>
@@
 <variant name="PC_Test_BOT" populate="no"/>
 </part>
-<part name="C42" library="Capacitors" library_urn="urn:adsk.eagle:library:13360199" deviceset="C-EU" device="0603" package3d_urn="urn:adsk.eagle:package:14720896/4" value="0.33u/16V">
-<variant name="Full_Assembly_BOT" populate="no"/>
-<variant name="PC_Test_BOT" populate="no"/>
-</part>
-<part name="C46" library="Capacitors" library_urn="urn:adsk.eagle:library:13360199" deviceset="C-EU" device="0603" package3d_urn="urn:adsk.eagle:package:14720896/4" value="0.33u/16V">
+<part name="C42" library="Capacitors" library_urn="urn:adsk.eagle:library:13360199" deviceset="C-EU" device="0603" package3d_urn="urn:adsk.eagle:package:14720896/4" value="0.33u/50V">
+<variant name="Full_Assembly_BOT" populate="no"/>
+<variant name="PC_Test_BOT" populate="no"/>
+</part>
+<part name="C46" library="Capacitors" library_urn="urn:adsk.eagle:library:13360199" deviceset="C-EU" device="0603" package3d_urn="urn:adsk.eagle:package:14720896/4" value="0.33u/50V">
 <variant name="Full_Assembly_BOT" populate="no"/>
 <variant name="PC_Test_BOT" populate="no"/>
@@
 balanced them and transmit all information to MasterBMS</text>
 <text x="135.89" y="-165.1" size="1.778" layer="97">https://github.com/701lab/SlaveBMS</text>
+<text x="-58.42" y="-96.52" size="1.778" layer="171">fail in 50V cap
+voltage rating</text>
+<text x="-60.96" y="-127" size="1.778" layer="171">fail in 50V cap
+voltage rating</text>
+<text x="66.04" y="20.32" size="1.778" layer="171">fail in 50V cap
+voltage rating</text>
+<text x="66.04" y="50.8" size="1.778" layer="171">fail in 50V cap
+voltage rating</text>
+<text x="27.94" y="71.12" size="1.778" layer="171">fail in 100V cap
+voltage rating</text>
 </plain>
 <instances>
