File: Slave BMS ESKD.sch (EAGLE design)
At the start: 152 parts, among them J1 S4B-PH-K, J12 MOLEX22-12-406205-7068, J2 S4B-PH-K, J3 S4B-PH-K, J4 S4B-PH-K, J5 S2B-PH-K, U1 BQ79606A-Q1-HTQFP|48|9VIA, X1 PESD2CAN, X2 PESD2CAN, X3 PESD2CAN, X4 PESD2CAN

Commit message: Some changes
I don't know
Parts:
- removed AVDD, VLDO, VSS: TEST_PAD-[1.27MM_SK], testing:TEST_PAD-[1.27MM_SK]
- removed BAT, CHN, CHP, CLN, CLP, FHN, FHP, FLN, FLP, REF, VC0, VC1, VC2, VC3, VC4, VC5, VC6: TEST_PAD-[1MM_SK], testing:TEST_PAD-[1MM_SK]
- removed BAT0, BAT1, BAT2, BAT3, BAT4, BAT5, BAT6: TEST_RING, testing:TEST_RING
- removed C54, C56: 2.2n, Capacitors:C-EU-K1206
- removed C55: 0.47u/16V, Capacitors:C-EU0603
- removed C57: 51p, Capacitors:C-EU0603
- removed C58, C59: 1nF, Capacitors:C-EU0603
- removed C72: 1u/16V, Capacitors:C-EU-K-X0603
- removed D13: GREEN, Semiconductor_devices:LED0805
- removed J1, J2, J3, J4: S4B-PH-K, con-jst-ph:S4B-PH-K
- removed J12: MOLEX22-12-406205-7068, commonly used connectors:MOLEX22-12-406205-7068
- removed J5: S2B-PH-K, con-jst-ph:S2B-PH-K
- removed JP4: 2x7, commonly used connectors:PINHD-2X7
- removed PROG+, PROG-: (no value), testing:SMD_PAD
- removed R68, R69, R70, R71, R72, R73: 10k, Resistors:R-EU0603
- removed R74: 100, 0.25W, Resistors:R-EU0603
- removed U$1: ESCD_CAP_EXT, ESCD:ESCD_CAP_EXT
- removed U$3: ESCD_RES_EXT, ESCD:ESCD_RES_EXT
- removed X1, X2, X3, X4: PESD2CAN, stmicroelectronics:PESD2CAN
- added C12, C15, C17, C19: 0.47u/16V, ESCD:ESCD_CAP
- added C14, C18: 1u/16V, ESCD:ESCD_CAP
- added D1: ESCD_LED, ESCD:ESCD_LED
- added D2, D3, D4, D5: SOT_23_TVS, ESCD:SOT_23_TVS
- added PAD1, PAD2: (no value), testing:SMD_PAD
- added R17: 10, 1/4W, ESCD:ESCD_RES
- added R18: 100, 0.25W, ESCD:ESCD_RES
- added R22: ESCD_RES, ESCD:ESCD_RES
- added R48: 10k, ESCD:ESCD_RES
- added R6: 47, ESCD:ESCD_RES
- C1, C2: value 0.33u/50V -> 0.1u/100V; device Capacitors:C-EU-K1206 -> ESCD:ESCD_CAP
- C10: value 2.2u/16V -> 0.47u/16V; device Capacitors:C-EU0603 -> ESCD:ESCD_CAP
- C11: value 2.2u/16V -> 1u/16V; device Capacitors:C-EU0603 -> ESCD:ESCD_CAP
- C13: value 2.2n -> 0.47u/16V; device Capacitors:C-EU-K1206 -> ESCD:ESCD_CAP
- C16: value 1u/16V -> 0.47u/16V; device Capacitors:C-EU0603 -> ESCD:ESCD_CAP
- C20: value 0.1u/100V -> ESCD_CAP; device Capacitors:C-EU-K1206 -> ESCD:ESCD_CAP
- C21: value 0.1u/100V -> 0.33u/50V; device Capacitors:C-EU-K1206 -> ESCD:ESCD_CAP
- C22, C24, C25: value 0.1u/100V -> 0.47u/16V; device Capacitors:C-EU-K1206 -> ESCD:ESCD_CAP
- C23: value 0.1u/100V -> 1u/16V; device Capacitors:C-EU-K1206 -> ESCD:ESCD_CAP
- C26, C27: value 0.47u/16V -> 0.33u/50V; device Capacitors:C-EU0603 -> ESCD:ESCD_CAP
- C28, C39, C52, C53, C7, C9: device Capacitors:C-EU0603 -> ESCD:ESCD_CAP
- C29: value 1u/16V -> 0.33u/50V; device Capacitors:C-EU-K0805 -> ESCD:ESCD_CAP
- C3, C4, C6: value 2.2u/16V -> 0.1u/100V; device Capacitors:C-EU0603 -> ESCD:ESCD_CAP
- C30: value 1u/16V -> ESCD_CAP; device Capacitors:C-EU-K0805 -> ESCD:ESCD_CAP
- C31: value 0.47u/16V -> 1nF; device Capacitors:C-EU0603 -> ESCD:ESCD_CAP
- C32: value 0.33u/50V -> 1nF; device Capacitors:C-EU0603 -> ESCD:ESCD_CAP
- C33: value 0.47u/16V -> 2.2u/16V; device Capacitors:C-EU0603 -> ESCD:ESCD_CAP
- C34, C37: value 2.2n -> 2.2u/16V; device Capacitors:C-EU-K1206 -> ESCD:ESCD_CAP
- C35, C8: value 51p -> 2.2u/16V; device Capacitors:C-EU0603 -> ESCD:ESCD_CAP
- C36: value 51p -> 0.33u/50V; device Capacitors:C-EU0603 -> ESCD:ESCD_CAP
- C38, C50, C51: value 2.2n -> 51p; device Capacitors:C-EU-K1206 -> ESCD:ESCD_CAP
- C40, C41: value 0.47u/16V -> 51p; device Capacitors:C-EU0603 -> ESCD:ESCD_CAP
- C42, C46: value 0.33u/50V -> 2.2n; device Capacitors:C-EU0603 -> ESCD:ESCD_CAP
- C43, C47, C48: value 0.47u/16V -> 2.2n; device Capacitors:C-EU0603 -> ESCD:ESCD_CAP
- C44, C45: value 1u/16V -> 2.2n; device Capacitors:C-EU-K0805 -> ESCD:ESCD_CAP
- C49: value 51p -> 2.2n; device Capacitors:C-EU0603 -> ESCD:ESCD_CAP
- C5: value 51p -> 0.1u/100V; device Capacitors:C-EU0603 -> ESCD:ESCD_CAP
- L1, L2, L3, L4: device Inductors:TDK_ACT45BIND_BOURNS_SRF4532-M -> ESCD:TDK_ACT45BIND_BOURNS_SRF4532-M
- R1: value 47, 0.25W -> 1k; device Resistors:R-EU1206 -> ESCD:ESCD_RES
- R10: value 10 -> ESCD_RES; device Resistors:R-EU0603 -> ESCD:ESCD_RES
- R11, R15, R16: value 10 -> 10, 1/4W; device Resistors:R-EU0603 -> ESCD:ESCD_RES
- R12, R13: value 43 -> 10, 1/4W; device Resistors:R-EU0603 -> ESCD:ESCD_RES
- R14: value 10k -> 10, 1/4W; device Resistors:R-EU0603 -> ESCD:ESCD_RES
- R19: value 1k -> ESCD_RES; device Resistors:R-EU0603 -> ESCD:ESCD_RES
- R2: value 100, 0.25W -> 47; device Resistors:R-EU0603 -> ESCD:ESCD_RES
- R20: value 100k -> ESCD_RES; device Resistors:R-EU0603 -> ESCD:ESCD_RES
- R21: value (none) -> 10k; device Resistors:R-EU-X0603 -> ESCD:ESCD_RES
- R23, R24, R25: value 47 -> ESCD_RES; device Resistors:R-EU0603 -> ESCD:ESCD_RES
- R26, R27, R29: value 47 -> 10k; device Resistors:R-EU0603 -> ESCD:ESCD_RES
- R28: value 47 -> 47, 0.25W; device Resistors:R-EU0603 -> ESCD:ESCD_RES
- R3: value 10k -> 47; device Resistors:R-EU0603 -> ESCD:ESCD_RES
- R30: value 10, 1/4W -> 10k; device Resistors:R-EU1210 -> ESCD:ESCD_RES
- R31, R32, R33, R34: value 10, 1/4W -> 43; device Resistors:R-EU1210 -> ESCD:ESCD_RES
- R35, R36: value 10, 1/4W -> 10; device Resistors:R-EU1210 -> ESCD:ESCD_RES
- R37, R38, R42: value 43 -> 10; device Resistors:R-EU0603 -> ESCD:ESCD_RES
- R39: value 10k -> 10; device Resistors:R-EU0603 -> ESCD:ESCD_RES
- R4, R5: value 10 -> 47; device Resistors:R-EU0603 -> ESCD:ESCD_RES
- R40, R41, R43, R47: device Resistors:R-EU0603 -> ESCD:ESCD_RES
- R44: value 1k -> 43; device Resistors:R-EU0603 -> ESCD:ESCD_RES
- R45, R46: value 10k -> 43; device Resistors:R-EU0603 -> ESCD:ESCD_RES
- R7, R8: value 43 -> 47; device Resistors:R-EU0603 -> ESCD:ESCD_RES
- R9: value 10k -> ESCD_RES; device Resistors:R-EU0603 -> ESCD:ESCD_RES
- U1: device texas Instrumets:BQ79606A-Q1-HTQFP|48|9VIA -> ESCD:BQ79606A-Q1-HTQFP|48|9VIA
Connections:
- removed net 125: C58.2, R46.1
- removed net 4: J4.4
- removed net CH1_N: C54.2, R41.2
- removed net CH1_P: C56.2, R40.2
- removed net CH2_N: C54.1, L4.2
- removed net CH2_P: C56.1, L4.1
- removed net CH_N: R41.1, R43.2, X4.1
- removed net CH_P: R40.1, R42.2, X4.2
- removed net COMH_N: C53.2, CHN.P$1, R39.1, R43.1, U1.COMHN
- removed net COMH_P: C52.2, CHP.P$1, R39.2, R42.1, U1.COMHP
- removed net COML_N: C36.2, CLN.P$1, R13.1, R9.1, U1.COMLN
- removed net COML_P: C35.2, CLP.P$1, R12.1, R9.2, U1.COMLP
- removed net FAULTH_N: C49.2, FHN.P$1, R14.1, R38.1, U1.FAULTHN
- removed net FAULTH_P: C39.2, FHP.P$1, R14.2, R37.1, U1.FAULTHP
- removed net FAULTL_N: C8.2, FLN.P$1, R3.1, R8.1, U1.FAULTLN
- removed net FAULTL_P: C5.2, FLP.P$1, R3.2, R7.1, U1.FAULTLP
- removed net FH1_N: C50.2, R16.2
- removed net FH1_P: C51.2, R15.2
- removed net FH2_N: C50.1, L3.2
- removed net FH2_P: C51.1, L3.1
- removed net FH_N: R16.1, R38.2, X3.1
- removed net FH_P: R15.1, R37.2, X3.2
- removed net GPIO6T1: J5.1, R20.1, R21.2
- removed net ISO_COMH_N: J3.4, L4.3
- removed net ISO_COMH_P: J3.3, L4.4
- removed net ISO_COML_N: J2.1, L2.4
- removed net ISO_COML_P: J2.2, L2.3
- removed net ISO_FAULTH_N: J3.2, L3.3
- removed net ISO_FAULTH_P: J3.1, L3.4
- removed net ISO_FAULTL_N: J2.3, L1.4
- removed net ISO_FAULTL_P: J2.4, L1.3
- removed net N$1: C57.2
- removed net N$23: R69.1
- removed net N$24: R68.1
- removed net N$28: D13.A, R44.1
- removed net N$8: J12-1.S
- removed net NFAULT: C59.2, J12-5.S, R45.1, U1.NFAULT
- removed net RX1: J12-3.S, R74.1
- removed net SB0: JP4.13, R36.1
- removed net SB1: JP4.11, R35.1
- removed net SB2: JP4.9, R34.1
- removed net SB3: JP4.7, R33.1
- removed net SB4: JP4.5, R32.1
- removed net SB5: JP4.3, R31.1
- removed net SB6: JP4.1, R30.1
- removed net WAKEUP: U1.WAKEUP
- new net CL1_N1: C42.2, R39.2
- new net CL1_P1: C43.2, R40.2
- new net CL2_N1: C42.1, L1.1
- new net CL2_P1: C43.1, L1.2
- new net CL_N1: D4.1, R39.1, R43.2
- new net CL_P1: D4.2, R40.1, R44.2
- new net CMH_N: C50.2, R43.1, R47.1, U1.COMHN
- new net CMH_P: C51.2, R44.1, R47.2, U1.COMHP
- new net CML_N: C38.2, R29.1, R31.1, U1.COMLN
- new net CML_P: C39.2, R29.2, R32.1, U1.COMLP
- new net FL1_N1: C44.2, R41.2
- new net FL1_P1: C45.2, R42.2
- new net FL2_N1: C44.1, L2.1
- new net FL2_P1: C45.1, L2.2
- new net FL_N1: R41.1, R45.2
- new net FL_P1: R42.1, R46.2
- new net FTH_N: C52.2, R45.1, R48.1, U1.FLTHN
- new net FTH_P: C53.2, R46.1, R48.2, U1.FLTHP
- new net FTL_N: C40.2, R30.1, R33.1, U1.FLTLN
- new net FTL_P: C41.2, R30.2, R34.1, U1.FLTLP
- new net N$12: L4.3
- new net N$14: L1.3
- new net N$15: L1.4
- new net N$16: L2.4
- new net N$17: L2.3
- new net N$2: D1.A, R1.1
- new net N$7: L4.4
- new net N$9: C31.2, R22.2, R26.1
- new net NFLT: C30.1, R27.1, U1.NFAULT
- new net WKP: C32.2, U1.WKP
- net AVDD: now also C7.1, R1.2; no longer AVDD.P$1, C6.1, R44.2
- net BAT: now also R18.1; no longer BAT.P$1, R2.1
- net BAT1: now also C3.2, C6.1, R16.1, R7.1; no longer BAT1.P$1, C24.1, C25.2, J4.3, JP4.12, R28.1
- net BAT2: now also C2.1, C6.2, R15.1, R6.1; no longer BAT2.P$1, C23.1, C24.2, J1.2, JP4.10, R27.1
- net BAT3: now also C2.2, C5.1, R14.1, R5.1; no longer BAT3.P$1, C22.1, C23.2, J4.2, JP4.8, R26.1
- net BAT4: now also C1.1, C5.2, R13.1, R4.1; no longer BAT4.P$1, C21.1, C22.2, J1.3, JP4.6, R25.1
- net BAT5: now also C1.2, C4.1, R12.1, R3.1; no longer BAT5.P$1, C20.1, C21.2, J4.1, JP4.4, R24.1
- net CB0: now also C19.1, C25.2, R17.2, U1.CB6; no longer C48.1, C55.2, R36.2
- net CB1: now also C19.2, C24.1, C29.1, R16.2; no longer C46.1, C47.1, C48.2, R35.2
- net CB2: now also C18.1, C24.2, C29.2, R15.2; no longer C45.1, C46.2, C47.2, R34.2
- net CB3: now also C18.2, C23.1, R14.2; no longer C44.1, C45.2, R33.2
- net CB4: now also C17.1, C23.2, C28.1, R13.2; no longer C42.1, C43.1, C44.2, R32.2
- net CB5: now also C17.2, C22.1, C28.2, R12.2; no longer C41.1, C42.2, C43.2, R31.2
- net CB6: now also C22.2, R11.2; no longer C41.2, R30.2, U1.CB6
- net CL1_N: now also C46.2, R35.2; no longer C37.2, R11.2
- net CL1_P: now also C47.2, R36.2; no longer C38.2, R10.2
- net CL2_N: now also C46.1, L3.1; no longer C37.1, L2.1
- net CL2_P: now also C47.1, L3.2; no longer C38.1, L2.2
- net CL_N: now also D2.1, R31.2, R35.1; no longer R11.1, R13.2, X1.2
- net CL_P: now also D2.2, R32.2, R36.1; no longer R10.1, R12.2, X1.1
- net DVDD: now also C34.1; no longer C10.1
- net FL1_N: now also C48.2, R37.2; no longer C13.2, R5.2
- net FL1_P: now also C49.2, R38.2; no longer C34.2, R4.2
- net FL2_N: now also C48.1, L4.1; no longer C13.1, L1.1
- net FL2_P: now also C49.1, L4.2; no longer C34.1, L1.2
- net FL_N: now also R33.2, R37.1; no longer R5.1, R8.2, X2.2
- net FL_P: now also R34.2, R38.1; no longer R4.1, R7.2, X2.1
- net GND: now also C20.2, C21.2, C3.1, C30.2, C31.1, C32.1, C33.2, C34.2, C35.2, C36.2, C37.2, C38.1, C41.1, C50.1, C51.1, C8.2, D1.K, D2.3, D3.3, D4.3, D5.3, PAD2.P, R17.1, R19.2, R20.2, R23.2, R24.2, R25.2, R8.1; no longer BAT0.P$1, C1.1, C10.2, C11.2, C2.2, C3.2, C35.1, C36.1, C4.2, C49.1, C5.1, C55.1, C57.1, C58.1, C59.1, C6.2, C72.2, C8.1, D13.C, J1.1, J12-6.S, J5.2, JP4.14, PROG-.P, R21.1, R29.1, R68.2, R69.2, R70.2, R71.2, R72.2, R73.2, VSS.P$1, X1.3, X2.3, X3.3, X4.3
- net GPIO1: now also C20.1, R10.2; no longer C16.2, R19.1
- net GPIO2: now also R23.1; no longer R73.1
- net GPIO3: now also R19.1; no longer R72.1
- net GPIO4: now also R24.1
- net GPIO5: now also R20.1
- net GPIO6: now also R25.1
- net LDOIN: now also R28.1; no longer R1.1
- net N$4: now also L3.3; no longer R71.1
- net N$5: now also R10.1, R9.1; no longer R19.2
- net N$6: now also L3.4; no longer R70.1
- net REF1: now also C9.1; no longer C4.1, REF.P$1
- net RX: now also R22.1; no longer R47.1, R74.2
- net TSREF: now also C8.1, R9.2; no longer C3.1, C72.1, R20.2
- net TX: now also R21.1; no longer J12-2.S
- net VC0: now also C12.1, C16.2, R8.2; no longer C33.1, C40.2, R29.2, VC0.P$1
- net VC1: now also C12.2, C15.1, C27.1, R7.2; no longer C31.1, C32.1, C33.2, R28.2, VC1.P$1
- net VC2: now also C11.1, C15.2, C27.2, R6.2; no longer C30.1, C31.2, C32.2, R27.2, VC2.P$1
- net VC3: now also C11.2, C14.1, R5.2; no longer C29.1, C30.2, R26.2, VC3.P$1
- net VC4: now also C10.1, C14.2, C26.1, R4.2; no longer C27.1, C28.1, C29.2, R25.2, VC4.P$1
- net VC5: now also C10.2, C13.1, C26.2, R3.2; no longer C26.1, C27.2, C28.2, R24.2, VC5.P$1
- net VC6: now also C13.2, R2.2; no longer C26.2, R23.2, VC6.P$1
- net VCC: now also C21.1, C36.1, C4.2, R11.1, R18.2, R2.1, R28.2; no longer BAT6.P$1, C1.2, C2.1, C20.2, J1.4, JP4.2, R1.2, R2.2, R23.1
- net VIO: now also C33.1, R21.2, R26.2, R27.2; no longer C11.1, J12-4.S, R45.2, R46.2, R47.2
- net VLDO: now also C35.1, C37.1; no longer C7.1, C9.1, VLDO.P$1
- net VPROG: now also PAD1.P; no longer PROG+.P
Other:
- note added: "1"
- note added: "10"
- note added: "11"
- note added: "12"
- note added: "13"
- note added: "2"
- note added: "3"
- note added: "4"
- note added: "5"
- note added: "6"
- note added: "7"
- note added: "8"
- note added: "9"
- note added: "BAT0"
- note added: "BAT1"
- note added: "BAT2"
- note added: "BAT3"
- note added: "BAT4"
- note added: "BAT5"
- note added: "BAT6"
- note added: "CMHN"
- note added: "CMHP"
- note added: "CMLN"
- note added: "CMLP"
- note added: "D2"
- note added: "D3"
- note added: "D4"
- note added: "D5"
- note added: "FTHN"
- note added: "FTHP"
- note added: "FTLN"
- note added: "FTLP"
- note added: "GND"
- note added: "NFLT"
- note added: "RX"
- note added: "TS1"
- note added: "TS2"
- note added: "TX"
- note added: "VCC"
- note added: "WKP"
- note added: "БГУИР, гр.721901"
- note added: "Вход"
- note added: "Выход"
- note added: "ГУИР.442226.001 Э3"
- note added: "Городко"
- note added: "Система мониторинга параметров аккумуляторных батарей"
- note added: "Схема электрическая принципиальная"
- note added: "Цепь"
- note added: "Яскевич"
- moved on the sheet: R21
